Commit message: UDの胴体部のURDFを記述した

File: config/youbot_base_only.urdf.xacro (robot description, xacro)
@@ -26,6 +26,4 @@
   <xacro:youbot_base name="base"/>
   <!-- base laser front -->
-  <xacro:hokuyo_urg04_laser name="base_laser_front" parent="base" ros_topic="base_scan" update_rate="10" min_angle="-1.57" max_angle="1.57">
-    <origin xyz="0.3 0 -0.03" rpy="0 0 0"/>
-  </xacro:hokuyo_urg04_laser>
+  <!-- The configuration of hokuyo_urg04_laser is moved to ud.urdf.xacro -->
 </robot>
