Commit message: 胴体部を下部と上部に分割した

File: config/ud.urdf.xacro (robot description, xacro)
@@ -6,8 +6,11 @@
        name="ud" >
   <xacro:include filename="$(find ubiquitous_display)/config/youbot_base_only.urdf.xacro" />
-  <property name="pillar_height" value="0.5"/>
+  <property name="bottom_pillar_height" value="0.2"/>
+  <property name="top_pillar_height" value="0.4"/>
   <property name="pillar_radius" value="0.01"/>
   <property name="pillar_offset_x" value="0.2"/>
   <property name="pillar_offset_y" value="0.07"/>
+  <property name="plate_len_x" value="0.5"/>
+  <property name="plate_len_y" value="0.2"/>
   <material name="black">
     <color rgba="0 0 0 1"/>
@@ -17,50 +20,99 @@
   </material>
   <!-- Body -->
-  <link name="pillars">
+  <!-- Bottom part -->
+  <link name="bottom_pillars">
     <visual>
       <geometry>
-        <cylinder length="${pillar_height}" radius="${pillar_radius}"/>
+        <cylinder length="${bottom_pillar_height}" radius="${pillar_radius}"/>
       </geometry>
-      <origin xyz="${pillar_offset_x} ${pillar_offset_y} ${pillar_height/2}"/>
+      <origin xyz="${pillar_offset_x} ${pillar_offset_y} ${bottom_pillar_height/2}"/>
       <material name="black"/>
     </visual>
     <visual>
       <geometry>
-        <cylinder length="${pillar_height}" radius="${pillar_radius}"/>
+        <cylinder length="${bottom_pillar_height}" radius="${pillar_radius}"/>
       </geometry>
-      <origin xyz="-${pillar_offset_x} ${pillar_offset_y} ${pillar_height/2}"/>
+      <origin xyz="-${pillar_offset_x} ${pillar_offset_y} ${bottom_pillar_height/2}"/>
       <material name="black"/>
     </visual>
     <visual>
       <geometry>
-        <cylinder length="${pillar_height}" radius="${pillar_radius}"/>
+        <cylinder length="${bottom_pillar_height}" radius="${pillar_radius}"/>
       </geometry>
-      <origin xyz="${pillar_offset_x} -${pillar_offset_y} ${pillar_height/2}"/>
+      <origin xyz="${pillar_offset_x} -${pillar_offset_y} ${bottom_pillar_height/2}"/>
       <material name="black"/>
     </visual>
     <visual>
       <geometry>
-        <cylinder length="${pillar_height}" radius="${pillar_radius}"/>
+        <cylinder length="${bottom_pillar_height}" radius="${pillar_radius}"/>
       </geometry>
-      <origin xyz="-${pillar_offset_x} -${pillar_offset_y} ${pillar_height/2}"/>
+      <origin xyz="-${pillar_offset_x} -${pillar_offset_y} ${bottom_pillar_height/2}"/>
       <material name="black"/>
     </visual>
   </link>
-  <joint name="base_to_pillars" type="fixed">
+  <joint name="base_to_bottom_pillars" type="fixed">
     <parent link="base_link"/>
-    <child link="pillars"/>
+    <child link="bottom_pillars"/>
+  </joint>
+  <link name="bottom_plate">
+    <visual>
+      <geometry>
+        <box size="${plate_len_x} ${plate_len_y} 0.01"/>
+      </geometry>
+      <material name="white"/>
+    </visual>
+  </link>
+  <joint name="bottom_pillars_to_bottom_plate" type="fixed">
+    <parent link="bottom_pillars"/>
+    <child link="bottom_plate"/>
+    <origin xyz="0 0 ${bottom_pillar_height}"/>
+  </joint>
+  <!-- Top part -->
+  <link name="top_pillars">
+    <visual>
+      <geometry>
+        <cylinder length="${top_pillar_height}" radius="${pillar_radius}"/>
+      </geometry>
+      <origin xyz="${pillar_offset_x} ${pillar_offset_y} ${top_pillar_height/2}"/>
+      <material name="black"/>
+    </visual>
+    <visual>
+      <geometry>
+        <cylinder length="${top_pillar_height}" radius="${pillar_radius}"/>
+      </geometry>
+      <origin xyz="-${pillar_offset_x} ${pillar_offset_y} ${top_pillar_height/2}"/>
+      <material name="black"/>
+    </visual>
+    <visual>
+      <geometry>
+        <cylinder length="${top_pillar_height}" radius="${pillar_radius}"/>
+      </geometry>
+      <origin xyz="${pillar_offset_x} -${pillar_offset_y} ${top_pillar_height/2}"/>
+      <material name="black"/>
+    </visual>
+    <visual>
+      <geometry>
+        <cylinder length="${top_pillar_height}" radius="${pillar_radius}"/>
+      </geometry>
+      <origin xyz="-${pillar_offset_x} -${pillar_offset_y} ${top_pillar_height/2}"/>
+      <material name="black"/>
+    </visual>
+  </link>
+  <joint name="bottom_plate_to_top_pillars" type="fixed">
+    <parent link="bottom_plate"/>
+    <child link="top_pillars"/>
   </joint>
   <link name="top_plate">
     <visual>
       <geometry>
-       <box size="0.4 0.14 0.01"/>
+        <box size="${plate_len_x} ${plate_len_y} 0.01"/>
       </geometry>
       <material name="white"/>
     </visual>
   </link>
-  <joint name="pillars_to_top_plate" type="fixed">
-    <parent link="pillars"/>
+  <joint name="top_pillars_to_top_plate" type="fixed">
+    <parent link="top_pillars"/>
     <child link="top_plate"/>
-    <origin xyz="0 0 ${pillar_height}"/>
+    <origin xyz="0 0 ${top_pillar_height}"/>
   </joint>
   <!-- base laser front -->

Commit message: Rename links and joints

File: config/ud.urdf.xacro (robot description, xacro)
@@ -21,5 +21,5 @@
   <!-- Body -->
   <!-- Bottom part -->
-  <link name="bottom_pillars">
+  <link name="bottom_pillars_link">
     <visual>
       <geometry>
@@ -51,9 +51,9 @@
     </visual>
   </link>
-  <joint name="base_to_bottom_pillars" type="fixed">
+  <joint name="base_to_bottom_pillars_joint" type="fixed">
     <parent link="base_link"/>
-    <child link="bottom_pillars"/>
+    <child link="bottom_pillars_link"/>
   </joint>
-  <link name="bottom_plate">
+  <link name="bottom_plate_link">
     <visual>
       <geometry>
@@ -63,11 +63,11 @@
     </visual>
   </link>
-  <joint name="bottom_pillars_to_bottom_plate" type="fixed">
-    <parent link="bottom_pillars"/>
-    <child link="bottom_plate"/>
+  <joint name="bottom_pillars_to_bottom_plate_joint" type="fixed">
+    <parent link="bottom_pillars_link"/>
+    <child link="bottom_plate_link"/>
     <origin xyz="0 0 ${bottom_pillar_height}"/>
   </joint>
   <!-- Top part -->
-  <link name="top_pillars">
+  <link name="top_pillars_link">
     <visual>
       <geometry>
@@ -99,9 +99,9 @@
     </visual>
   </link>
-  <joint name="bottom_plate_to_top_pillars" type="fixed">
-    <parent link="bottom_plate"/>
-    <child link="top_pillars"/>
+  <joint name="bottom_plate_to_top_pillars_joint" type="fixed">
+    <parent link="bottom_plate_link"/>
+    <child link="top_pillars_link"/>
   </joint>
-  <link name="top_plate">
+  <link name="top_plate_link">
     <visual>
       <geometry>
@@ -111,7 +111,7 @@
     </visual>
   </link>
-  <joint name="top_pillars_to_top_plate" type="fixed">
-    <parent link="top_pillars"/>
-    <child link="top_plate"/>
+  <joint name="top_pillars_to_top_plate_joint" type="fixed">
+    <parent link="top_pillars_link"/>
+    <child link="top_plate_link"/>
     <origin xyz="0 0 ${top_pillar_height}"/>
   </joint>

Commit message: Hokuyoの親をbottom plateに変更した

File: config/ud.urdf.xacro (robot description, xacro)
@@ -13,4 +13,6 @@
   <property name="plate_len_x" value="0.5"/>
   <property name="plate_len_y" value="0.2"/>
+  <property name="hokuyo_offset_x" value="0.25"/>
+  <property name="hokuyo_offset_z" value="0.04"/>
   <material name="black">
     <color rgba="0 0 0 1"/>
@@ -117,6 +119,6 @@
   </joint>
   <!-- base laser front -->
-  <xacro:hokuyo_urg04_laser name="base_laser_front" parent="base" ros_topic="base_scan" update_rate="10" min_angle="-1.57" max_angle="1.57">
-    <origin xyz="0.25 0 0.22" rpy="0 0 0"/>
+  <xacro:hokuyo_urg04_laser name="base_laser_front" parent="bottom_plate" ros_topic="base_scan" update_rate="10" min_angle="-1.57" max_angle="1.57">
+    <origin xyz="${hokuyo_offset_x} 0 ${hokuyo_offset_z}" rpy="0 0 0"/>
   </xacro:hokuyo_urg04_laser>
 </robot>

Commit message: plateのoriginを上面に配置した

File: config/ud.urdf.xacro (robot description, xacro)
@@ -13,6 +13,7 @@
   <property name="plate_len_x" value="0.5"/>
   <property name="plate_len_y" value="0.2"/>
+  <property name="plate_len_z" value="0.01"/>
   <property name="hokuyo_offset_x" value="0.25"/>
-  <property name="hokuyo_offset_z" value="0.04"/>
+  <property name="hokuyo_offset_z" value="0.035"/>
   <material name="black">
     <color rgba="0 0 0 1"/>
@@ -60,6 +61,7 @@
     <visual>
       <geometry>
-        <box size="${plate_len_x} ${plate_len_y} 0.01"/>
+        <box size="${plate_len_x} ${plate_len_y} ${plate_len_z}"/>
       </geometry>
+      <origin xyz="0 0 -${plate_len_z/2}"/>
       <material name="white"/>
     </visual>
@@ -108,6 +110,7 @@
     <visual>
       <geometry>
-        <box size="${plate_len_x} ${plate_len_y} 0.01"/>
+        <box size="${plate_len_x} ${plate_len_y} ${plate_len_z}"/>
       </geometry>
+      <origin xyz="0 0 -${plate_len_z/2}"/>
       <material name="white"/>
     </visual>
