Commit message: UDのURDFを実際の寸法に合わせて修正した．

File: urdf/ud.urdf.xacro (robot description, xacro)
@@ -7,14 +7,18 @@
   <xacro:include filename="$(find ubiquitous_display)/urdf/youbot_base_only.urdf.xacro" />
   <!-- Definition of various sizes -->
-  <property name="bottom_pillar_height" value="0.2"/>
-  <property name="top_pillar_height" value="0.4"/>
+  <property name="bottom_pillar_height" value="0.1"/>
+  <property name="middle_pillar_height" value="0.157"/>
+  <property name="top_pillar_height" value="0.435"/>
   <property name="pillar_radius" value="0.01"/>
-  <property name="pillar_offset_x" value="0.2"/>
-  <property name="pillar_offset_y" value="0.07"/>
+  <property name="pillar_offset_x" value="0.21"/>
+  <property name="pillar_offset_y" value="0.06"/>
   <property name="plate_len_x" value="0.5"/>
   <property name="plate_len_y" value="0.2"/>
-  <property name="plate_len_z" value="0.01"/>
+  <property name="plate_len_z" value="0.004"/>
+  <property name="bar_len_x" value="0.18"/>
+  <property name="bar_len_y" value="0.02"/>
+  <property name="bar_len_z" value="0.02"/>
   <property name="hokuyo_offset_x" value="0.25"/>
-  <property name="hokuyo_offset_z" value="0.035"/>
+  <property name="hokuyo_offset_z" value="0.037"/>
   <!-- Definition of colors -->
   <material name="black">
@@ -68,4 +72,39 @@
       <material name="white"/>
     </visual>
+    <visual>
+      <geometry>
+        <box size="${bar_len_x} ${bar_len_y} ${bar_len_z}"/>
+      </geometry>
+      <origin xyz="0.20 0.025 ${bar_len_z/2}"/>
+     <material name="gray" />
+    </visual>
+    <visual>
+      <geometry>
+        <box size="${bar_len_x} ${bar_len_y} ${bar_len_z}"/>
+      </geometry>
+      <origin xyz="0.20 -0.025 ${bar_len_z/2}"/>
+     <material name="gray" />
+    </visual>
+    <visual>
+      <geometry>
+        <box size="${bar_len_x} ${bar_len_y} ${bar_len_z}"/>
+      </geometry>
+      <origin xyz="-0.20 0.025 ${bar_len_z/2}"/>
+     <material name="gray" />
+    </visual>
+    <visual>
+      <geometry>
+        <box size="${bar_len_x} ${bar_len_y} ${bar_len_z}"/>
+      </geometry>
+      <origin xyz="-0.20 0.025 ${bar_len_z/2}"/>
+     <material name="gray" />
+    </visual>
+    <visual>
+      <geometry>
+        <box size="${bar_len_x} ${bar_len_y} ${bar_len_z}"/>
+      </geometry>
+      <origin xyz="-0.20 -0.025 ${bar_len_z/2}"/>
+     <material name="gray" />
+    </visual>
   </link>
   <joint name="bottom_pillars_to_bottom_plate_joint" type="fixed">
@@ -74,4 +113,53 @@
     <origin xyz="0 0 ${bottom_pillar_height}"/>
   </joint>
+ <!-- Middle part -->
+  <link name="middle_pillars_link">
+    <visual>
+      <geometry>
+        <cylinder length="${middle_pillar_height}" radius="${pillar_radius}"/>
+      </geometry>
+      <origin xyz="${pillar_offset_x} ${pillar_offset_y} ${middle_pillar_height/2}"/>
+      <material name="black"/>
+    </visual>
+    <visual>
+      <geometry>
+        <cylinder length="${middle_pillar_height}" radius="${pillar_radius}"/>
+      </geometry>
+      <origin xyz="-${pillar_offset_x} ${pillar_offset_y} ${middle_pillar_height/2}"/>
+      <material name="black"/>
+    </visual>
+    <visual>
+      <geometry>
+        <cylinder length="${middle_pillar_height}" radius="${pillar_radius}"/>
+      </geometry>
+      <origin xyz="${pillar_offset_x} -${pillar_offset_y} ${middle_pillar_height/2}"/>
+      <material name="black"/>
+    </visual>
+    <visual>
+      <geometry>
+        <cylinder length="${middle_pillar_height}" radius="${pillar_radius}"/>
+      </geometry>
+      <origin xyz="-${pillar_offset_x} -${pillar_offset_y} ${middle_pillar_height/2}"/>
+      <material name="black"/>
+    </visual>
+  </link>
+  <joint name="bottom_plate_to_middle_pillars_joint" type="fixed">
+    <parent link="bottom_plate_link"/>
+    <child link="middle_pillars_link"/>
+  </joint>
+  <link name="middle_plate_link">
+    <visual>
+      <geometry>
+        <box size="${plate_len_x} ${plate_len_y} ${plate_len_z}"/>
+      </geometry>
+      <origin xyz="0 0 -${plate_len_z/2}"/>
+      <material name="white"/>
+    </visual>
+  </link>
+  <joint name="bottom_plate_to_middle_plate_joint" type="fixed">
+    <parent link="bottom_plate_link"/>
+    <child link="middle_plate_link"/>
+    <origin xyz="0 0 ${middle_pillar_height}"/>
+  </joint>
   <!-- Top part -->
   <link name="top_pillars_link">
@@ -105,6 +193,6 @@
     </visual>
   </link>
-  <joint name="bottom_plate_to_top_pillars_joint" type="fixed">
-    <parent link="bottom_plate_link"/>
+  <joint name="middle_plate_to_top_pillars_joint" type="fixed">
+    <parent link="middle_plate_link"/>
     <child link="top_pillars_link"/>
   </joint>

Commit message: 2台目のLRFを追加した．

File: urdf/ud.urdf.xacro (robot description, xacro)
@@ -215,3 +215,7 @@
     <origin xyz="${hokuyo_offset_x} 0 ${hokuyo_offset_z}" rpy="0 0 0"/>
   </xacro:hokuyo_urg04_laser>
+  <!-- base laser rear -->
+  <xacro:hokuyo_urg04_laser name="base_laser_rear" parent="bottom_plate" ros_topic="base_scan" update_rate="10" min_angle="-1.57" max_angle="1.57">
+    <origin xyz="-${hokuyo_offset_x} 0 ${hokuyo_offset_z}" rpy="0 0 3.14"/>
+  </xacro:hokuyo_urg04_laser>
 </robot>

Commit message: Fix the parent of the middle_plate

File: urdf/ud.urdf.xacro (robot description, xacro)
@@ -157,6 +157,6 @@
     </visual>
   </link>
-  <joint name="bottom_plate_to_middle_plate_joint" type="fixed">
-    <parent link="bottom_plate_link"/>
+  <joint name="middle_pillars_to_middle_plate_joint" type="fixed">
+    <parent link="middle_pillars_link"/>
     <child link="middle_plate_link"/>
     <origin xyz="0 0 ${middle_pillar_height}"/>

Commit message: Use body.urdf in ud.urdf

File: urdf/ud.urdf.xacro (robot description, xacro)
@@ -6,216 +6,19 @@
        name="ud" >
   <xacro:include filename="$(find ubiquitous_display)/urdf/youbot_base_only.urdf.xacro" />
-  <!-- Definition of various sizes -->
-  <property name="bottom_pillar_height" value="0.1"/>
-  <property name="middle_pillar_height" value="0.157"/>
-  <property name="top_pillar_height" value="0.435"/>
-  <property name="pillar_radius" value="0.01"/>
-  <property name="pillar_offset_x" value="0.21"/>
-  <property name="pillar_offset_y" value="0.06"/>
-  <property name="plate_len_x" value="0.5"/>
-  <property name="plate_len_y" value="0.2"/>
-  <property name="plate_len_z" value="0.004"/>
-  <property name="bar_len_x" value="0.18"/>
-  <property name="bar_len_y" value="0.02"/>
-  <property name="bar_len_z" value="0.02"/>
-  <property name="hokuyo_offset_x" value="0.25"/>
+  <xacro:include filename="$(find ubiquitous_display)/urdf/body.urdf.xacro" />
+  <property name="hokuyo_offset_x" value="-0.05"/>
   <property name="hokuyo_offset_z" value="0.037"/>
-  <!-- Definition of colors -->
-  <material name="black">
-    <color rgba="0 0 0 1"/>
-  </material>
-  <material name="white">
-    <color rgba="1 1 1 1"/>
-  </material>
-  <!-- Body -->
-  <!-- Bottom part -->
-  <link name="bottom_pillars_link">
-    <visual>
-      <geometry>
-        <cylinder length="${bottom_pillar_height}" radius="${pillar_radius}"/>
-      </geometry>
-      <origin xyz="${pillar_offset_x} ${pillar_offset_y} ${bottom_pillar_height/2}"/>
-      <material name="black"/>
-    </visual>
-    <visual>
-      <geometry>
-        <cylinder length="${bottom_pillar_height}" radius="${pillar_radius}"/>
-      </geometry>
-      <origin xyz="-${pillar_offset_x} ${pillar_offset_y} ${bottom_pillar_height/2}"/>
-      <material name="black"/>
-    </visual>
-    <visual>
-      <geometry>
-        <cylinder length="${bottom_pillar_height}" radius="${pillar_radius}"/>
-      </geometry>
-      <origin xyz="${pillar_offset_x} -${pillar_offset_y} ${bottom_pillar_height/2}"/>
-      <material name="black"/>
-    </visual>
-    <visual>
-      <geometry>
-        <cylinder length="${bottom_pillar_height}" radius="${pillar_radius}"/>
-      </geometry>
-      <origin xyz="-${pillar_offset_x} -${pillar_offset_y} ${bottom_pillar_height/2}"/>
-      <material name="black"/>
-    </visual>
-  </link>
-  <joint name="base_to_bottom_pillars_joint" type="fixed">
+  <joint name="youbot_to_body_joint" type="fixed">
+    <ogirin xyz="0 0 0" rpy="0 0 0"/>
     <parent link="base_link"/>
     <child link="bottom_pillars_link"/>
   </joint>
-  <link name="bottom_plate_link">
-    <visual>
-      <geometry>
-        <box size="${plate_len_x} ${plate_len_y} ${plate_len_z}"/>
-      </geometry>
-      <origin xyz="0 0 -${plate_len_z/2}"/>
-      <material name="white"/>
-    </visual>
-    <visual>
-      <geometry>
-        <box size="${bar_len_x} ${bar_len_y} ${bar_len_z}"/>
-      </geometry>
-      <origin xyz="0.20 0.025 ${bar_len_z/2}"/>
-     <material name="gray" />
-    </visual>
-    <visual>
-      <geometry>
-        <box size="${bar_len_x} ${bar_len_y} ${bar_len_z}"/>
-      </geometry>
-      <origin xyz="0.20 -0.025 ${bar_len_z/2}"/>
-     <material name="gray" />
-    </visual>
-    <visual>
-      <geometry>
-        <box size="${bar_len_x} ${bar_len_y} ${bar_len_z}"/>
-      </geometry>
-      <origin xyz="-0.20 0.025 ${bar_len_z/2}"/>
-     <material name="gray" />
-    </visual>
-    <visual>
-      <geometry>
-        <box size="${bar_len_x} ${bar_len_y} ${bar_len_z}"/>
-      </geometry>
-      <origin xyz="-0.20 0.025 ${bar_len_z/2}"/>
-     <material name="gray" />
-    </visual>
-    <visual>
-      <geometry>
-        <box size="${bar_len_x} ${bar_len_y} ${bar_len_z}"/>
-      </geometry>
-      <origin xyz="-0.20 -0.025 ${bar_len_z/2}"/>
-     <material name="gray" />
-    </visual>
-  </link>
-  <joint name="bottom_pillars_to_bottom_plate_joint" type="fixed">
-    <parent link="bottom_pillars_link"/>
-    <child link="bottom_plate_link"/>
-    <origin xyz="0 0 ${bottom_pillar_height}"/>
-  </joint>
- <!-- Middle part -->
-  <link name="middle_pillars_link">
-    <visual>
-      <geometry>
-        <cylinder length="${middle_pillar_height}" radius="${pillar_radius}"/>
-      </geometry>
-      <origin xyz="${pillar_offset_x} ${pillar_offset_y} ${middle_pillar_height/2}"/>
-      <material name="black"/>
-    </visual>
-    <visual>
-      <geometry>
-        <cylinder length="${middle_pillar_height}" radius="${pillar_radius}"/>
-      </geometry>
-      <origin xyz="-${pillar_offset_x} ${pillar_offset_y} ${middle_pillar_height/2}"/>
-      <material name="black"/>
-    </visual>
-    <visual>
-      <geometry>
-        <cylinder length="${middle_pillar_height}" radius="${pillar_radius}"/>
-      </geometry>
-      <origin xyz="${pillar_offset_x} -${pillar_offset_y} ${middle_pillar_height/2}"/>
-      <material name="black"/>
-    </visual>
-    <visual>
-      <geometry>
-        <cylinder length="${middle_pillar_height}" radius="${pillar_radius}"/>
-      </geometry>
-      <origin xyz="-${pillar_offset_x} -${pillar_offset_y} ${middle_pillar_height/2}"/>
-      <material name="black"/>
-    </visual>
-  </link>
-  <joint name="bottom_plate_to_middle_pillars_joint" type="fixed">
-    <parent link="bottom_plate_link"/>
-    <child link="middle_pillars_link"/>
-  </joint>
-  <link name="middle_plate_link">
-    <visual>
-      <geometry>
-        <box size="${plate_len_x} ${plate_len_y} ${plate_len_z}"/>
-      </geometry>
-      <origin xyz="0 0 -${plate_len_z/2}"/>
-      <material name="white"/>
-    </visual>
-  </link>
-  <joint name="middle_pillars_to_middle_plate_joint" type="fixed">
-    <parent link="middle_pillars_link"/>
-    <child link="middle_plate_link"/>
-    <origin xyz="0 0 ${middle_pillar_height}"/>
-  </joint>
-  <!-- Top part -->
-  <link name="top_pillars_link">
-    <visual>
-      <geometry>
-        <cylinder length="${top_pillar_height}" radius="${pillar_radius}"/>
-      </geometry>
-      <origin xyz="${pillar_offset_x} ${pillar_offset_y} ${top_pillar_height/2}"/>
-      <material name="black"/>
-    </visual>
-    <visual>
-      <geometry>
-        <cylinder length="${top_pillar_height}" radius="${pillar_radius}"/>
-      </geometry>
-      <origin xyz="-${pillar_offset_x} ${pillar_offset_y} ${top_pillar_height/2}"/>
-      <material name="black"/>
-    </visual>
-    <visual>
-      <geometry>
-        <cylinder length="${top_pillar_height}" radius="${pillar_radius}"/>
-      </geometry>
-      <origin xyz="${pillar_offset_x} -${pillar_offset_y} ${top_pillar_height/2}"/>
-      <material name="black"/>
-    </visual>
-    <visual>
-      <geometry>
-        <cylinder length="${top_pillar_height}" radius="${pillar_radius}"/>
-      </geometry>
-      <origin xyz="-${pillar_offset_x} -${pillar_offset_y} ${top_pillar_height/2}"/>
-      <material name="black"/>
-    </visual>
-  </link>
-  <joint name="middle_plate_to_top_pillars_joint" type="fixed">
-    <parent link="middle_plate_link"/>
-    <child link="top_pillars_link"/>
-  </joint>
-  <link name="top_plate_link">
-    <visual>
-      <geometry>
-        <box size="${plate_len_x} ${plate_len_y} ${plate_len_z}"/>
-      </geometry>
-      <origin xyz="0 0 -${plate_len_z/2}"/>
-      <material name="white"/>
-    </visual>
-  </link>
-  <joint name="top_pillars_to_top_plate_joint" type="fixed">
-    <parent link="top_pillars_link"/>
-    <child link="top_plate_link"/>
-    <origin xyz="0 0 ${top_pillar_height}"/>
-  </joint>
   <!-- base laser front -->
-  <xacro:hokuyo_urg04_laser name="base_laser_front" parent="bottom_plate" ros_topic="base_scan" update_rate="10" min_angle="-1.57" max_angle="1.57">
+  <xacro:hokuyo_urg04_laser name="base_laser_front" parent="front_laser_adjuster" ros_topic="base_scan" update_rate="10" min_angle="-1.57" max_angle="1.57">
     <origin xyz="${hokuyo_offset_x} 0 ${hokuyo_offset_z}" rpy="0 0 0"/>
   </xacro:hokuyo_urg04_laser>
   <!-- base laser rear -->
-  <xacro:hokuyo_urg04_laser name="base_laser_rear" parent="bottom_plate" ros_topic="base_scan" update_rate="10" min_angle="-1.57" max_angle="1.57">
-    <origin xyz="-${hokuyo_offset_x} 0 ${hokuyo_offset_z}" rpy="0 0 3.14"/>
+  <xacro:hokuyo_urg04_laser name="base_laser_rear" parent="rear_laser_adjuster" ros_topic="base_scan" update_rate="10" min_angle="-1.57" max_angle="1.57">
+    <origin xyz="${hokuyo_offset_x} 0 ${hokuyo_offset_z}" rpy="0 0 0"/>
   </xacro:hokuyo_urg04_laser>
 </robot>

Commit message: Integrate pantilt into ud.

File: urdf/ud.urdf.xacro (robot description, xacro)
@@ -7,4 +7,5 @@
   <xacro:include filename="$(find ubiquitous_display)/urdf/youbot_base_only.urdf.xacro" />
   <xacro:include filename="$(find ubiquitous_display)/urdf/body.urdf.xacro" />
+  <xacro:include filename="$(find ubiquitous_display)/urdf/pantilt.urdf.xacro" />
   <property name="hokuyo_offset_x" value="-0.05"/>
   <property name="hokuyo_offset_z" value="0.037"/>
@@ -13,4 +14,9 @@
     <parent link="base_link"/>
     <child link="bottom_pillars_link"/>
+  </joint>
+  <joint name="body_to_pantilt_joint" type="fixed">
+    <ogirin xyz="0 0 0" rpy="0 0 0"/>
+    <parent link="top_plate_link"/>
+    <child link="ud_pt_base_link"/>
   </joint>
   <!-- base laser front -->
