Commit message: modify joint name

File: urdf/pantilt.urdf.xacro (robot description, xacro)
@@ -54,5 +54,6 @@
       <origin xyz="0 0 0" rpy="0 0 0" />
     </joint>
-    <joint name="${name}pan_joint" type="revolute">
+    <!--name of pan_joint and tilt_joint depend pantilt.yaml-->
+    <joint name="pan_joint" type="revolute">
       <parent link="${name}box_link"/>
       <child link="${name}plate_link"/>
@@ -61,5 +62,5 @@
       <limit lower="0" upper="2" effort="1" velocity="1"/>
     </joint>
-    <joint name="${name}tilt_joint" type="revolute">
+    <joint name="tilt_joint" type="revolute">
       <parent link="${name}plate_link"/>
       <child link="${name}projector_link"/>

Commit message: Indentation

File: urdf/pantilt.urdf.xacro (robot description, xacro)
@@ -1,8 +1,8 @@
 <?xml version="1.0"?>
 <robot xmlns:sensor="http://playerstage.sourceforge.net/gazebo/xmlschema/#sensor"
-       xmlns:controller="http://playerstage.sourceforge.net/gazebo/xmlschema/#controller"
-       xmlns:interface="http://playerstage.sourceforge.net/gazebo/xmlschema/#interface"
-       xmlns:xacro="http://playerstage.sourceforge.net/gazebo/xmlschema/#interface"
-       name="pantilt" >
+  xmlns:controller="http://playerstage.sourceforge.net/gazebo/xmlschema/#controller"
+  xmlns:interface="http://playerstage.sourceforge.net/gazebo/xmlschema/#interface"
+  xmlns:xacro="http://playerstage.sourceforge.net/gazebo/xmlschema/#interface"
+  name="pantilt" >
   <property name="base_to_box_height" value="0.065"/>
   <property name="box_to_proj_height" value="0.17"/>
@@ -23,29 +23,29 @@
     </link>
     <link name="${name}box_link" >
-     <visual>
-       <origin xyz="0 0 0" rpy="0 0 0" />
-       <geometry>
-         <box size="0.07 0.085 0.065" />
-       </geometry>
-       <material name="red"/>
-     </visual>
+      <visual>
+        <origin xyz="0 0 0" rpy="0 0 0" />
+        <geometry>
+          <box size="0.07 0.085 0.065" />
+        </geometry>
+        <material name="red"/>
+      </visual>
     </link>
     <link name="${name}plate_link">
-        <visual>
-       <origin xyz="0 0 0" rpy="0 0 0" />
-       <geometry>
-         <box size="0.35 0.095 0.003" />
-       </geometry>
-       <material name="green"/>
-     </visual>
+      <visual>
+        <origin xyz="0 0 0" rpy="0 0 0" />
+        <geometry>
+          <box size="0.35 0.095 0.003" />
+        </geometry>
+        <material name="green"/>
+      </visual>
     </link>
     <link name="${name}projector_link">
-         <visual>
-       <origin xyz="0 0 0" rpy="0 0 0" />
-       <geometry>
-         <box size="0.24 0.17 0.07" />
-       </geometry>
-       <material name="white"/>
-     </visual>
+      <visual>
+        <origin xyz="0 0 0" rpy="0 0 0" />
+        <geometry>
+          <box size="0.24 0.17 0.07" />
+        </geometry>
+        <material name="white"/>
+      </visual>
     </link>
     <joint name="${name}base_joint" type="fixed">

Commit message: Change the color name from white to gray to prevent confliction

File: urdf/pantilt.urdf.xacro (robot description, xacro)
@@ -16,5 +16,5 @@
     <color rgba="0.0 0.7 0.7 1.0" />
   </material>
-  <material name="white" >
+  <material name="gray" >
     <color rgba="0.7 0.7 0.7 1.0" />
   </material>
@@ -46,5 +46,5 @@
           <box size="0.24 0.17 0.07" />
         </geometry>
-        <material name="white"/>
+        <material name="gray"/>
       </visual>
     </link>
